File: TreeOrnament.sch (KiCad schematic (older format))
At the start: 0 parts

Commit message: Add some LEDs.
Parts:
- added D? (x8): LED, symbol LED
- added J?: USB_B_Micro, symbol USB_B_Micro
- added R? (x4): 56, symbol R
Connections:
- new net: D?.2 (A), R?.2 (x4)
- new net: D?.1 (K), D?.2 (A) (x4)
- new net +5V: J?.1 (VBUS), R?.1, R?.1, R?.1, R?.1
- new net GND: D?.1 (K), D?.1 (K), D?.1 (K), D?.1 (K), J?.5 (GND), J?.6 (Shield)
Changed lines of the file:
@@
 LIBS:valves
 LIBS:myLibrary
+LIBS:TreeOrnament-cache
 EELAYER 25 0
 EELAYER END
@@
 Comment4 ""
 $EndDescr
+$Comp
+L USB_B_Micro J?
+U 1 1 59EFEC98
+P 1500 1400
+F 0 "J?" H 1300 1850 50  0000 L CNN
+F 1 "USB_B_Micro" H 1300 1750 50  0000 L CNN
+F 2 "" H 1650 1350 50  0001 C CNN
+F 3 "" H 1650 1350 50  0001 C CNN
+	1    1500 1400
+	1    0    0    -1
+$EndComp
+$Comp
+L GND #PWR?
+U 1 1 59EFECD5
+P 1500 2000
+F 0 "#PWR?" H 1500 1750 50  0001 C CNN
+F 1 "GND" H 1500 1850 50  0000 C CNN
+F 2 "" H 1500 2000 50  0001 C CNN
+F 3 "" H 1500 2000 50  0001 C CNN
+	1    1500 2000
+	1    0    0    -1
+$EndComp
+$Comp
+L +5V #PWR?
+U 1 1 59EFED06
+P 2000 1000
+F 0 "#PWR?" H 2000 850 50  0001 C CNN
+F 1 "+5V" H 2000 1140 50  0000 C CNN
+F 2 "" H 2000 1000 50  0001 C CNN
+F 3 "" H 2000 1000 50  0001 C CNN
+	1    2000 1000
+	1    0    0    -1
+$EndComp
+Wire Wire Line
+	1800 1200 5700 1200
+Wire Wire Line
+	2000 1200 2000 1000
+Wire Wire Line
+	1500 1800 1500 2000
+Wire Wire Line
+	1400 1800 1400 1900
+Wire Wire Line
+	1400 1900 4900 1900
+Connection ~ 1500 1900
+$Comp
+L R R?
+U 1 1 59EFED4B
+P 3000 1450
+F 0 "R?" V 3080 1450 50  0000 C CNN
+F 1 "56" V 3000 1450 50  0000 C CNN
+F 2 "" V 2930 1450 50  0001 C CNN
+F 3 "" H 3000 1450 50  0001 C CNN
+	1    3000 1450
+	1    0    0    -1
+$EndComp
+$Comp
+L LED D?
+U 1 1 59EFED7C
+P 2450 1700
+F 0 "D?" H 2450 1800 50  0000 C CNN
+F 1 "LED" H 2450 1600 50  0000 C CNN
+F 2 "" H 2450 1700 50  0001 C CNN
+F 3 "" H 2450 1700 50  0001 C CNN
+	1    2450 1700
+	1    0    0    -1
+$EndComp
+$Comp
+L LED D?
+U 1 1 59EFED9B
+P 2850 1700
+F 0 "D?" H 2850 1800 50  0000 C CNN
+F 1 "LED" H 2850 1600 50  0000 C CNN
+F 2 "" H 2850 1700 50  0001 C CNN
+F 3 "" H 2850 1700 50  0001 C CNN
+	1    2850 1700
+	1    0    0    -1
+$EndComp
+Wire Wire Line
+	3000 1200 3000 1300
+Connection ~ 2000 1200
+Wire Wire Line
+	3000 1600 3000 1700
+Wire Wire Line
+	2700 1700 2600 1700
+Wire Wire Line
+	2300 1700 2200 1700
+Wire Wire Line
+	2200 1700 2200 1900
+$Comp
+L R R?
+U 1 1 59EFEE1B
+P 3900 1450
+F 0 "R?" V 3980 1450 50  0000 C CNN
+F 1 "56" V 3900 1450 50  0000 C CNN
+F 2 "" V 3830 1450 50  0001 C CNN
+F 3 "" H 3900 1450 50  0001 C CNN
+	1    3900 1450
+	1    0    0    -1
+$EndComp
+$Comp
+L LED D?
+U 1 1 59EFEE4E
+P 3350 1700
+F 0 "D?" H 3350 1800 50  0000 C CNN
+F 1 "LED" H 3350 1600 50  0000 C CNN
+F 2 "" H 3350 1700 50  0001 C CNN
+F 3 "" H 3350 1700 50  0001 C CNN
+	1    3350 1700
+	1    0    0    -1
+$EndComp
+$Comp
+L LED D?
+U 1 1 59EFEE7A
+P 3750 1700
+F 0 "D?" H 3750 1800 50  0000 C CNN
+F 1 "LED" H 3750 1600 50  0000 C CNN
+F 2 "" H 3750 1700 50  0001 C CNN
+F 3 "" H 3750 1700 50  0001 C CNN
+	1    3750 1700
+	1    0    0    -1
+$EndComp
+Wire Wire Line
+	3900 1200 3900 1300
+Connection ~ 3000 1200
+Wire Wire Line
+	3900 1600 3900 1700
+Wire Wire Line
+	3600 1700 3500 1700
+Wire Wire Line
+	3200 1700 3100 1700
+Wire Wire Line
+	3100 1700 3100 1900
+Connection ~ 2200 1900
+$Comp
+L LED D?
+U 1 1 59EFEF28
+P 4250 1700
+F 0 "D?" H 4250 1800 50  0000 C CNN
+F 1 "LED" H 4250 1600 50  0000 C CNN
+F 2 "" H 4250 1700 50  0001 C CNN
+F 3 "" H 4250 1700 50  0001 C CNN
+	1    4250 1700
+	1    0    0    -1
+$EndComp
+$Comp
+L LED D?
+U 1 1 59EFEF58
+P 4650 1700
+F 0 "D?" H 4650 1800 50  0000 C CNN
+F 1 "LED" H 4650 1600 50  0000 C CNN
+F 2 "" H 4650 1700 50  0001 C CNN
+F 3 "" H 4650 1700 50  0001 C CNN
+	1    4650 1700
+	1    0    0    -1
+$EndComp
+$Comp
+L R R?
+U 1 1 59EFEF89
+P 4800 1450
+F 0 "R?" V 4880 1450 50  0000 C CNN
+F 1 "56" V 4800 1450 50  0000 C CNN
+F 2 "" V 4730 1450 50  0001 C CNN
+F 3 "" H 4800 1450 50  0001 C CNN
+	1    4800 1450
+	1    0    0    -1
+$EndComp
+Wire Wire Line
+	4800 1200 4800 1300
+Connection ~ 3900 1200
+Wire Wire Line
+	4800 1600 4800 1700
+Wire Wire Line
+	4500 1700 4400 1700
+Wire Wire Line
+	4100 1700 4000 1700
+Wire Wire Line
+	4000 1700 4000 1900
+Connection ~ 3100 1900
+$Comp
+L LED D?
+U 1 1 59EFF04E
+P 5150 1700
+F 0 "D?" H 5150 1800 50  0000 C CNN
+F 1 "LED" H 5150 1600 50  0000 C CNN
+F 2 "" H 5150 1700 50  0001 C CNN
+F 3 "" H 5150 1700 50  0001 C CNN
+	1    5150 1700
+	1    0    0    -1
+$EndComp
+$Comp
+L LED D?
+U 1 1 59EFF087
+P 5550 1700
+F 0 "D?" H 5550 1800 50  0000 C CNN
+F 1 "LED" H 5550 1600 50  0000 C CNN
+F 2 "" H 5550 1700 50  0001 C CNN
+F 3 "" H 5550 1700 50  0001 C CNN
+	1    5550 1700
+	1    0    0    -1
+$EndComp
+$Comp
+L R R?
+U 1 1 59EFF0C1
+P 5700 1450
+F 0 "R?" V 5780 1450 50  0000 C CNN
+F 1 "56" V 5700 1450 50  0000 C CNN
+F 2 "" V 5630 1450 50  0001 C CNN
+F 3 "" H 5700 1450 50  0001 C CNN
+	1    5700 1450
+	1    0    0    -1
+$EndComp
+Wire Wire Line
+	5700 1200 5700 1300
+Connection ~ 4800 1200
+Wire Wire Line
+	5700 1600 5700 1700
+Wire Wire Line
+	5400 1700 5300 1700
+Wire Wire Line
+	5000 1700 4900 1700
+Wire Wire Line
+	4900 1700 4900 1900
+Connection ~ 4000 1900
 $EndSCHEMATC
