File: TreeOrnament.sch (KiCad schematic (older format))
At the start: 32 parts, among them J1 USB_B_Micro

Commit message: Change resistor value from 150 to 1k.
Parts:
- R1, R10, R11, R12, R13, R14, R2, R3, R4, R5, R6, R7, R8, R9: value 150 -> 1k
Changed lines of the file:
@@
 Sheet 1 1
 Title "Christmas Tree Ornament"
-Date "2017-11-02"
-Rev "1.1"
+Date "2017-11-25"
+Rev "1.2"
 Comp "Patrick Pelletier"
 Comment1 ""
@@
 P 3000 1450
 F 0 "R2" V 3080 1450 50  0000 C CNN
-F 1 "150" V 3000 1450 50  0000 C CNN
+F 1 "1k" V 3000 1450 50  0000 C CNN
 F 2 "myLibrary:R_Axial_DIN0204_L3.6mm_D1.6mm_P5.08mm_Horizontal" V 2930 1450 50  0001 C CNN
 F 3 "" H 3000 1450 50  0001 C CNN
@@
 P 3900 1450
 F 0 "R4" V 3980 1450 50  0000 C CNN
-F 1 "150" V 3900 1450 50  0000 C CNN
+F 1 "1k" V 3900 1450 50  0000 C CNN
 F 2 "myLibrary:R_Axial_DIN0204_L3.6mm_D1.6mm_P5.08mm_Horizontal" V 3830 1450 50  0001 C CNN
 F 3 "" H 3900 1450 50  0001 C CNN
@@
 P 4800 1450
 F 0 "R6" V 4880 1450 50  0000 C CNN
-F 1 "150" V 4800 1450 50  0000 C CNN
+F 1 "1k" V 4800 1450 50  0000 C CNN
 F 2 "myLibrary:R_Axial_DIN0204_L3.6mm_D1.6mm_P5.08mm_Horizontal" V 4730 1450 50  0001 C CNN
 F 3 "" H 4800 1450 50  0001 C CNN
@@
 P 5700 1450
 F 0 "R8" V 5780 1450 50  0000 C CNN
-F 1 "150" V 5700 1450 50  0000 C CNN
+F 1 "1k" V 5700 1450 50  0000 C CNN
 F 2 "myLibrary:R_Axial_DIN0204_L3.6mm_D1.6mm_P5.08mm_Horizontal" V 5630 1450 50  0001 C CNN
 F 3 "" H 5700 1450 50  0001 C CNN
@@
 P 6600 1450
 F 0 "R10" V 6680 1450 50  0000 C CNN
-F 1 "150" V 6600 1450 50  0000 C CNN
+F 1 "1k" V 6600 1450 50  0000 C CNN
 F 2 "myLibrary:R_Axial_DIN0204_L3.6mm_D1.6mm_P5.08mm_Horizontal" V 6530 1450 50  0001 C CNN
 F 3 "" H 6600 1450 50  0001 C CNN
@@
 P 7500 1450
 F 0 "R12" V 7580 1450 50  0000 C CNN
-F 1 "150" V 7500 1450 50  0000 C CNN
+F 1 "1k" V 7500 1450 50  0000 C CNN
 F 2 "myLibrary:R_Axial_DIN0204_L3.6mm_D1.6mm_P5.08mm_Horizontal" V 7430 1450 50  0001 C CNN
 F 3 "" H 7500 1450 50  0001 C CNN
@@
 P 8400 1450
 F 0 "R14" V 8480 1450 50  0000 C CNN
-F 1 "150" V 8400 1450 50  0000 C CNN
+F 1 "1k" V 8400 1450 50  0000 C CNN
 F 2 "myLibrary:R_Axial_DIN0204_L3.6mm_D1.6mm_P5.08mm_Horizontal" V 8330 1450 50  0001 C CNN
 F 3 "" H 8400 1450 50  0001 C CNN
@@
 P 2600 1450
 F 0 "R1" V 2680 1450 50  0000 C CNN
-F 1 "150" V 2600 1450 50  0000 C CNN
+F 1 "1k" V 2600 1450 50  0000 C CNN
 F 2 "myLibrary:R_Axial_DIN0204_L3.6mm_D1.6mm_P5.08mm_Horizontal" V 2530 1450 50  0001 C CNN
 F 3 "" H 2600 1450 50  0001 C CNN
@@
 P 3500 1450
 F 0 "R3" V 3580 1450 50  0000 C CNN
-F 1 "150" V 3500 1450 50  0000 C CNN
+F 1 "1k" V 3500 1450 50  0000 C CNN
 F 2 "myLibrary:R_Axial_DIN0204_L3.6mm_D1.6mm_P5.08mm_Horizontal" V 3430 1450 50  0001 C CNN
 F 3 "" H 3500 1450 50  0001 C CNN
@@
 P 4400 1450
 F 0 "R5" V 4480 1450 50  0000 C CNN
-F 1 "150" V 4400 1450 50  0000 C CNN
+F 1 "1k" V 4400 1450 50  0000 C CNN
 F 2 "myLibrary:R_Axial_DIN0204_L3.6mm_D1.6mm_P5.08mm_Horizontal" V 4330 1450 50  0001 C CNN
 F 3 "" H 4400 1450 50  0001 C CNN
@@
 P 5300 1450
 F 0 "R7" V 5380 1450 50  0000 C CNN
-F 1 "150" V 5300 1450 50  0000 C CNN
+F 1 "1k" V 5300 1450 50  0000 C CNN
 F 2 "myLibrary:R_Axial_DIN0204_L3.6mm_D1.6mm_P5.08mm_Horizontal" V 5230 1450 50  0001 C CNN
 F 3 "" H 5300 1450 50  0001 C CNN
@@
 P 6200 1450
 F 0 "R9" V 6280 1450 50  0000 C CNN
-F 1 "150" V 6200 1450 50  0000 C CNN
+F 1 "1k" V 6200 1450 50  0000 C CNN
 F 2 "myLibrary:R_Axial_DIN0204_L3.6mm_D1.6mm_P5.08mm_Horizontal" V 6130 1450 50  0001 C CNN
 F 3 "" H 6200 1450 50  0001 C CNN
@@
 P 7100 1450
 F 0 "R11" V 7180 1450 50  0000 C CNN
-F 1 "150" V 7100 1450 50  0000 C CNN
+F 1 "1k" V 7100 1450 50  0000 C CNN
 F 2 "myLibrary:R_Axial_DIN0204_L3.6mm_D1.6mm_P5.08mm_Horizontal" V 7030 1450 50  0001 C CNN
 F 3 "" H 7100 1450 50  0001 C CNN
@@
 P 8000 1450
 F 0 "R13" V 8080 1450 50  0000 C CNN
-F 1 "150" V 8000 1450 50  0000 C CNN
+F 1 "1k" V 8000 1450 50  0000 C CNN
 F 2 "myLibrary:R_Axial_DIN0204_L3.6mm_D1.6mm_P5.08mm_Horizontal" V 7930 1450 50  0001 C CNN
 F 3 "" H 8000 1450 50  0001 C CNN
